Commit message: Added files for mujoco adaptation

File: low-level/resources/robots/b1z1/urdf_mujoco/b1z1 (copy).urdf (robot description, URDF)
Before this commit: robot b1z1_description, 29 links, 28 joints
Links:
- link FL_calf: geometry collision box size=0.35 0.04 0.05; visual mesh filename=../meshes_new/calf.stl scale=1 1 1
- link FL_hip: geometry visual mesh filename=../meshes_new/hip.stl scale=1 1 1
- link FL_thigh: geometry collision box size=0.35 0.05 0.08; visual mesh filename=../meshes_new/thigh.stl scale=1 1 1
- link FR_calf: geometry collision box size=0.35 0.04 0.05; visual mesh filename=../meshes_new/calf.stl scale=1 1 1
- link FR_hip: geometry visual mesh filename=../meshes_new/hip.stl scale=1 1 1
- link FR_thigh: geometry collision box size=0.35 0.05 0.08; visual mesh filename=../meshes_new/thigh_mirror.stl scale=1 1 1
- link RL_calf: geometry collision box size=0.35 0.04 0.05; visual mesh filename=../meshes_new/calf.stl scale=1 1 1
- link RL_hip: geometry visual mesh filename=../meshes_new/hip.stl scale=1 1 1
- link RL_thigh: geometry collision box size=0.35 0.05 0.08; visual mesh filename=../meshes_new/thigh.stl scale=1 1 1
- link RR_calf: geometry collision box size=0.35 0.04 0.05; visual mesh filename=../meshes_new/calf.stl scale=1 1 1
- link RR_hip: geometry visual mesh filename=../meshes_new/hip.stl scale=1 1 1
- link RR_thigh: geometry collision box size=0.35 0.05 0.08; visual mesh filename=../meshes_new/thigh_mirror.stl scale=1 1 1
- link gripperMover: geometry collision mesh filename=../meshes_new/z1_GripperMover.stl scale=1 1 1; visual mesh filename=../meshes_new/z1_GripperMover.stl scale=1 1 1
- link gripperStator: geometry collision mesh filename=../meshes_new/z1_GripperStator.stl scale=1 1 1; visual mesh filename=../meshes_new/z1_GripperStator.stl scale=1 1 1
- link link00: geometry collision cylinder length=0.03 radius=0.0325; visual mesh filename=../meshes_new/z1_Link00.stl scale=1 1 1
- link link01: geometry visual mesh filename=../meshes_new/z1_Link01.stl scale=1 1 1
- link link02: geometry collision cylinder length=0.051 radius=0.0325; collision cylinder length=0.102 radius=0.02
- link link03: geometry collision cylinder length=0.059 radius=0.0325; collision cylinder length=0.116 radius=0.02
- link link04: geometry collision cylinder length=0.073 radius=0.0325; visual mesh filename=../meshes_new/z1_Link04.stl scale=1 1 1
- link link05: geometry visual mesh filename=../meshes_new/z1_Link05.stl scale=1 1 1
- link link06: geometry collision cylinder length=0.051 radius=0.0325; visual mesh filename=../meshes_new/z1_Link06.stl scale=1 1 1
- link trunk: geometry collision box size=0.647 0.3 0.15; visual mesh filename=../meshes_new/trunk.stl scale=1 1 1
Joints:
- joint base_static_joint: origin xyz=0.3 0 0.09>> rpy=0 0 0 -> xyz=0.3 0 0.09 rpy=0 0 0
